File: mp3-player.kicad_pcb (KiCad board)
At the start: 4 copper layers, 55 x 47 mm, 120 parts, among them J1 JST_PH_BATT_CONN, J3 MSD-4-A, J5 USB4215-03-A, J6 Conn_01x06_Pin, J7 AudioJack3, Q2 2N7002, SW2 SW_MEC_5E, SW3 SW_MEC_5E, SW4 SW_MEC_5E, SW5 SW_Push_Shielded, SW6 SW_Push_Shielded, SW9 EG1213, U1 RP2350_60QFN, U10 W25Q32JVSS, U2 MCP73832-2-OT, U3 MCP6001-OT, U4 LM66100DCK, U5 PCM5101A, U6 TPA6139A2PWR, U7 LM66100DCK, U8 TPL730F33-5TR, U9 TPL730F33-5TR, Y1 ABM8-272-T3

Commit message: production version 0.1
Parts:
- removed R13: 10k, user_footprints:R_0402_1005Metric_NoSilk
- added R40: 10k, user_footprints:R_0402_1005Metric_NoSilk, F.Cu at (142.4, 69.3)
- added R41: 10k, user_footprints:R_0402_1005Metric_NoSilk, F.Cu at (137.2, 66.2)
- added R42: 10k, user_footprints:R_0402_1005Metric_NoSilk, F.Cu at (142.4, 70.5)
- added R43: 10k, user_footprints:R_0402_1005Metric_NoSilk, F.Cu at (140.5, 64.8)
- moved C34 5.69 mm to (134.4, 90.6)
- moved C33 5.68 mm to (140.0, 91.7)
- moved R37 1.76 mm to (128.8, 94.6)
- moved R38 1.39 mm to (126.7, 94.6), turned to 90 degrees
- moved C38 1.10 mm to (141.5, 89.2)
- moved C27 0.72 mm to (136.7, 91.2), turned to -90 degrees
- moved C28 0.56 mm to (137.1, 81.3)
- moved C29 0.56 mm to (137.1, 80.3)
- moved BOOTSEL 0.40 mm to (143.6, 73.4)
- moved C36 0.40 mm to (136.0, 93.7)
- moved C37 0.40 mm to (140.0, 93.7)
- moved R15 0.40 mm to (137.5, 93.2)
- moved R16 0.40 mm to (138.5, 93.2)
- moved C32 0.18 mm to (140.0, 90.6)
- renumbered SW4 to SW2, SW2 to SW4
Routing:
- net GND: track 126.8 -> 118.9 mm, vias 66 -> 75
- net /GPIO5: track 15.2 -> 20.2 mm, vias 1 -> 2
- net +3V3: track 59.1 -> 62.4 mm, vias 24 -> 26
- net /GPIO7: track 14.0 -> 17.2 mm
- net VBUS: track 3.66 -> 0.96 mm
- net /GPIO6: track 15.9 -> 18.4 mm
- net /V_IN: track 33.5 -> 31.8 mm
- net /GPIO4: track 18.4 -> 20.1 mm
- net Net-(J5-CC1): track 2.00 -> 3.69 mm
- net /GPIO26_ADC0: track 24.1 -> 23.0 mm
- net Net-(U6-CP): track 3.69 -> 4.62 mm
- net Net-(J5-CC2): track 3.28 -> 4.19 mm
- net /GPIO27_ADC1: track 20.0 -> 20.7 mm
- net Net-(U6-CN): track 3.52 -> 2.96 mm
Other:
- board text added: "Check"
- board text added: "MiniMusicBox v0.1"
- board text added: "Polarity!"
- board text removed: "+"
- board text removed: "-"

Commit message: cleaned project files, added readme
Routing:
- net /OUT_L: track 4.67 -> 2.82 mm
- net GND: track 118.9 -> 119.5 mm
Other:
- board text added: "To change: center board in plane move side buttons through hole usb-c test points power draw fix? better battery management? header pins attatched to useful nets power button: when held down, sets the enable pins to high, but can only be pulled low by mcu (SR latch)"
