File: mp3-player.kicad_sch (KiCad schematic)
At the start: 120 parts, among them J1 JST_PH_BATT_CONN, J3 MSD-4-A, J4 SM03B-SRSS-TB, J5 USB4215-03-A, J6 Conn_01x06_Pin, J7 AudioJack3, Q2 2N7002, SW1 SW_Push, SW2 SW_MEC_5E, SW3 SW_MEC_5E, SW4 SW_MEC_5E, SW5 SW_Push_Shielded, SW6 SW_Push_Shielded, SW9 EG1213, U1 RP2350_60QFN, U10 W25Q32JVSS, U2 MCP73832-2-OT, U3 MCP6001-OT, U4 LM66100DCK, U5 PCM5101A, U6 TPA6139A2PWR, U7 LM66100DCK, U8 TPL730F33-5TR, U9 TPL730F33-5TR, Y1 ABM8-272-T3

Commit message: production version 0.1
Parts:
- removed R13: 10k, user_footprints:R_0402_1005Metric_NoSilk, symbol Device:R
- added R40, R41, R42, R43: 10k, user_footprints:R_0402_1005Metric_NoSilk, symbol Device:R
- renumbered SW4 to SW2, SW2 to SW4
Connections:
- net +3V3: now also R40.1, R41.1, R42.1, R43.1
- net GPIO4: now also R42.2
- net GPIO5: now also R43.2
- net GPIO6: now also R40.2
- net GPIO7: now also R41.2
Other:
- note removed: "mosfet to stop idle power drainage is it necessary?"
- note removed: "place 0.1u cap as close to power and ground pins as possible"
- moved on the sheet: C50, J3, J5, R17, R18, U3

Commit message: cleaned project files, added readme
Parts:
- added SW10: EG1213, user_footprints:OS102011MA1QN1_CNK, symbol UserSymbols:EG1213
Connections:
- net GND: now also SW10.3, SW10.SH
- net V_IN: now also SW10.1; no longer U8.3 (EN), U9.3 (EN)
- new net LDO_EN: SW10.2, U8.3 (EN), U9.3 (EN)
